File: pcb/pcb.kicad_sch (KiCad schematic)
At the start: 66 parts, among them IC1 W25Q16JVUXIQ, IC2 RP2040, IC3 AD8403ARUZ1-REEL, IC4 DS4432U+, IC5 XC6222D331MR-G, J1 USB_C_Receptacle, K1 G3VM-31WR_TR05_, Y2 ABM10AIG-12.000MHZ-2Z-T

Commit message: Update pcb
Parts:
- removed IC2: RP2040, RP2040:QFN40P700X700X90-57N-D, symbol RP2040:RP2040
- removed IC5: XC6222D331MR-G, XC6222D331MR-G:SOT95P280X130-5N, symbol XC6222D331MR-G:XC6222D331MR-G
- removed Y2: ABM10AIG-12.000MHZ-2Z-T, ABM10AIG-12.000MHZ-2Z-T:ABM10AIG, symbol ABM10AIG-12_000MHZ-2Z-T:ABM10AIG-12.000MHZ-2Z-T
- added IC5: LP38690SD-3.3_NOPB, LP38690SD-3.3_NOPB:SON95P300X300X80-7N, symbol LP38690SD-3_3_NOPB:LP38690SD-3.3_NOPB
- added IC6: RP2040, RP2040:QFN40P700X700X90-57N-D, symbol RP2040:RP2040
- added Y1: Crystal_GND24, Crystal:Crystal_SMD_2520-4Pin_2.5x2.0mm, symbol Device:Crystal_GND24
- C1, C11, C3: footprint Capacitor_SMD:C_0201_0603Metric -> Capacitor_SMD:C_0402_1005Metric; LCSC C610030 -> C412453
- C10, C12, C13, C14, C17, C18, C4, C5, C6, C7, C8, C9: footprint Capacitor_SMD:C_0201_0603Metric -> Capacitor_SMD:C_0402_1005Metric; LCSC C5259862 -> C394158
- C15, C16: footprint Capacitor_SMD:C_0201_0603Metric -> Capacitor_SMD:C_0402_1005Metric; LCSC C396694 -> C161495
- C2: value 2.2u -> 1u; footprint Capacitor_SMD:C_0201_0603Metric -> Capacitor_SMD:C_0402_1005Metric; LCSC C5240383 -> C412453
- IC1: LCSC C2843335 -> (none)
- IC3: LCSC C652779 -> (none)
- IC4: LCSC C2679620 -> (none)
- R1, R2: footprint Resistor_SMD:R_0201_0603Metric -> Resistor_SMD:R_0402_1005Metric; LCSC C2484262 -> C102938
- R10, R9: footprint Resistor_SMD:R_0201_0603Metric -> Resistor_SMD:R_0402_1005Metric; LCSC C2991673 -> C144716
- R3, R5: footprint Resistor_SMD:R_0201_0603Metric -> Resistor_SMD:R_0402_1005Metric; LCSC C162776 -> C705665
- R4: footprint Resistor_SMD:R_0201_0603Metric -> Resistor_SMD:R_0402_1005Metric; LCSC C253350 -> C2991755
- R6, R7: footprint Resistor_SMD:R_0201_0603Metric -> Resistor_SMD:R_0402_1005Metric; LCSC C100142 -> C138073
- R8: footprint Resistor_SMD:R_0201_0603Metric -> Resistor_SMD:R_0402_1005Metric; LCSC C850675 -> C163462
Connections:
- net +1V1: now also IC6.23 (DVDD_1), IC6.45 (VREG_VOUT), IC6.50 (DVDD_2)
- net +3V3: now also IC5.4 (OUT), IC5.5 (SNS), IC6.1 (IOVDD_1), IC6.10 (IOVDD_2), IC6.22 (IOVDD_3), IC6.33 (IOVDD_4), IC6.42 (IOVDD_5), IC6.43 (ADC_AVDD), IC6.44 (VREG_VIN), IC6.48 (USB_VDD), IC6.49 (IOVDD_6)
- net 3DS_TP255_IRDA: now also IC6.34 (GPIO22)
- net 3DS_TP52_POWER: now also IC6.27 (GPIO16)
- net 3DS_TP55_HOME: now also IC6.18 (GPIO15)
- net 3DS_TP58_WIFI: now also IC6.28 (GPIO17)
- net 3DS_TP80_START: now also IC6.17 (GPIO14)
- net 3DS_TP81_SELECT: now also IC6.16 (GPIO13)
- net 3DS_TP82_R: now also IC6.15 (GPIO12)
- net 3DS_TP83_L: now also IC6.14 (GPIO11)
- net 3DS_TP85_UP: now also IC6.29 (GPIO18)
- net 3DS_TP86_X: now also IC6.13 (GPIO10)
- net 3DS_TP87_LEFT: now also IC6.32 (GPIO21)
- net 3DS_TP88_Y: now also IC6.9 (GPIO7)
- net 3DS_TP89_A: now also IC6.12 (GPIO9)
- net 3DS_TP90_RIGHT: now also IC6.30 (GPIO19)
- net 3DS_TP91_DOWN: now also IC6.31 (GPIO20)
- net 3DS_TP92_B: now also IC6.11 (GPIO8)
- net GND: now also IC5.2 (GND_1), IC5.7 (GND_2), IC6.19 (TESTEN), IC6.57 (GND), Y1.2, Y1.4
- net I2C_SCL: now also IC6.3 (GPIO1)
- net I2C_SDA: now also IC6.2 (GPIO0)
- net POTS_SHDN: now also IC6.6 (GPIO4)
- net QSPI_SCLK: now also IC6.52 (QSPI_SCLK)
- net QSPI_SD0: now also IC6.53 (QSPI_SD0)
- net QSPI_SD1: now also IC6.55 (QSPI_SD1)
- net QSPI_SD2: now also IC6.54 (QSPI_SD2)
- net QSPI_SD3: now also IC6.51 (QSPI_SD3)
- net QSPI_SS: now also IC6.56 (QSPI_SS_N)
- net RELAY_A: now also IC6.8 (GPIO6)
- net SPI_CS: now also IC6.7 (GPIO5)
- net SPI_SCK: now also IC6.4 (GPIO2)
- net SPI_TX: now also IC6.5 (GPIO3)
- net USB_D+: now also IC6.47 (USB_DP)
- net USB_D-: now also IC6.46 (USB_DM)
- net XIN: now also IC6.20 (XIN), Y1.3
- net XOUT: now also IC6.21 (XOUT)
- net at C1.1, D1.1 (K), D2.1 (K): now also IC5.1 (IN_1), IC5.6 (IN_2)
- net at C15.1, R5.2: now also Y1.1
- net at TP4.1: now also IC6.25 (SWDIO)
- net at TP3.1: now also IC6.24 (SWCLK)

Commit message: Update PCB
Parts:
- removed TP3, TP4: TestPoint, TestPoint:TestPoint_Pad_D1.0mm, symbol Connector:TestPoint
- added D3: LED, LED_SMD:LED_0402_1005Metric, symbol Device:LED
- added FPC1: THD0515-24CL-SN, THD0515-24CL-SN:FPC-SMD_24P-P0.50_THD0515-24CL-SN, symbol THD0515-24CL-SN:THD0515-24CL-SN
- added J2: Conn_01x03_Socket, Connector_PinSocket_2.54mm:PinSocket_1x03_P2.54mm_Vertical, symbol Connector:Conn_01x03_Socket
- added R11: 91, Resistor_SMD:R_0402_1005Metric, symbol Device:R
Connections:
- net GND: now also J2.1 (Pin_1), R11.2
- net at IC6.24 (SWCLK): now also J2.2 (Pin_2)
- net at IC6.25 (SWDIO): now also J2.3 (Pin_3)
- net at IC6.37 (GPIO25): now also D3.2 (A)
- new net: D3.1 (K), R11.1
- no-connect marks 22 -> 21
Changed lines of the file:
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@@
   (no_connect (at 166.37 146.05))
   (no_connect (at 265.43 81.28))
-  (no_connect (at 265.43 88.9))
   (no_connect (at 45.72 82.55))
   (no_connect (at 45.72 64.77))
@@
     (stroke (width 0) (type default))
   )
-  (wire (pts (xy 245.11 147.32) (xy 245.11 129.54))
+  (wire (pts (xy 245.11 129.54) (xy 245.11 154.94))
     (stroke (width 0) (type default))
   )
@@
     (stroke (width 0) (type default))
   )
-  (wire (pts (xy 247.65 142.24) (xy 247.65 129.54))
-    (stroke (width 0) (type default))
-  )
   (wire (pts (xy 48.26 43.18) (xy 45.72 43.18))
     (stroke (width 0) (type default))
@@
     (stroke (width 0) (type default))
   )
+  (wire (pts (xy 265.43 88.9) (xy 271.78 88.9))
+    (stroke (width 0) (type default))
+  )
   (wire (pts (xy 166.37 153.67) (xy 167.64 153.67))
     (stroke (width 0) (type default))
@@
     (stroke (width 0) (type default))
   )
+  (wire (pts (xy 247.65 129.54) (xy 247.65 154.94))
+    (stroke (width 0) (type default))
+  )
   (wire (pts (xy 252.73 21.59) (xy 252.73 24.13))
     (stroke (width 0) (type default))
@@
     )
   )
+  (symbol (lib_id "THD0515-24CL-SN:THD0515-24CL-SN") (at 200.66 30.48 0) (unit 1)
+    (in_bom yes) (on_board yes) (dnp no) (fields_autoplaced)
+    (property "Reference" "FPC1" (at 209.55 28.575 0)
+      (effects (font (size 1.27 1.27)) (justify left))
+    )
+    (property "Value" "THD0515-24CL-SN" (at 209.55 31.115 0)
+      (effects (font (size 1.27 1.27)) (justify left))
+    )
+    (property "Footprint" "THD0515-24CL-SN:FPC-SMD_24P-P0.50_THD0515-24CL-SN" (at 200.66 71.12 0)
+      (effects (font (size 1.27 1.27)) hide)
+    )
+    (property "Datasheet" "https://lcsc.com/product-detail/FFC-FPC-Flat-Flexible-Connectors_THD-THD0515-24CL-SN_C283150.html" (at 200.66 73.66 0)
+      (effects (font (size 1.27 1.27)) hide)
+    )
+    (property "LCSC Part" "C283150" (at 200.66 76.2 0)
+      (effects (font (size 1.27 1.27)) hide)
+    )
+    (pin "1")
+    (pin "10")
+    (pin "11")
+    (pin "12")
+    (pin "13")
+    (pin "14")
+    (pin "15")
+    (pin "16")
+    (pin "17")
+    (pin "18")
+    (pin "19")
+    (pin "2")
+    (pin "20")
+    (pin "21")
+    (pin "22")
+    (pin "23")
+    (pin "24")
+    (pin "25")
+    (pin "26")
+    (pin "3")
+    (pin "4")
+    (pin "5")
+    (pin "6")
+    (pin "7")
+    (pin "8")
+    (pin "9")
+    (instances
+      (project "pcb"
+        (path "/20bda546-3b72-48f2-b51c-b61a4edfe0c6"
+          (reference "FPC1") (unit 1)
+        )
+      )
+    )
+  )
   (symbol (lib_id "Connector:TestPoint") (at 175.26 36.83 270) (unit 1)
     (in_bom yes) (on_board yes) (dnp no) (fields_autoplaced)
@@
     )
   )
+  (symbol (lib_id "Connector:Conn_01x03_Socket") (at 245.11 160.02 90) (mirror x) (unit 1)
+    (in_bom yes) (on_board yes) (dnp no) (fields_autoplaced)
+    (property "Reference" "J2" (at 245.11 162.56 90)
+      (effects (font (size 1.27 1.27)))
+    )
+    (property "Value" "Conn_01x03_Socket" (at 245.11 165.1 90)
+      (effects (font (size 1.27 1.27)))
+    )
+    (property "Footprint" "Connector_PinSocket_2.54mm:PinSocket_1x03_P2.54mm_Vertical" (at 245.11 160.02 0)
+      (effects (font (size 1.27 1.27)) hide)
+    )
+    (property "Datasheet" "~" (at 245.11 160.02 0)
+      (effects (font (size 1.27 1.27)) hide)
+    )
+    (pin "1")
+    (pin "2")
+    (pin "3")
+    (instances
+      (project "pcb"
+        (path "/20bda546-3b72-48f2-b51c-b61a4edfe0c6"
+          (reference "J2") (unit 1)
+        )
+      )
+    )
+  )
   (symbol (lib_id "power:GND") (at 175.26 104.14 90) (unit 1)
     (in_bom yes) (on_board yes) (dnp no) (fields_autoplaced)
@@
     )
   )
+  (symbol (lib_id "power:GND") (at 287.02 88.9 90) (unit 1)
+    (in_bom yes) (on_board yes) (dnp no) (fields_autoplaced)
+    (property "Reference" "#PWR026" (at 293.37 88.9 0)
+      (effects (font (size 1.27 1.27)) hide)
+    )
+    (property "Value" "GND" (at 290.83 89.535 90)
+      (effects (font (size 1.27 1.27)) (justify right))
+    )
+    (property "Footprint" "" (at 287.02 88.9 0)
+      (effects (font (size 1.27 1.27)) hide)
+    )
+    (property "Datasheet" "" (at 287.02 88.9 0)
+      (effects (font (size 1.27 1.27)) hide)
+    )
+    (pin "1")
+    (instances
+      (project "pcb"
+        (path "/19e8f276-6a71-4fad-b0cb-92febe4a4ffd"
+          (reference "#PWR026") (unit 1)
+        )
+      )
+      (project "pcb"
+        (path "/20bda546-3b72-48f2-b51c-b61a4edfe0c6"
+          (reference "#PWR010") (unit 1)
+        )
+      )
+    )
+  )
   (symbol (lib_id "power:GND") (at 78.74 106.68 90) (unit 1)
     (in_bom yes) (on_board yes) (dnp no) (fields_autoplaced)
@@
     )
   )
-  (symbol (lib_id "Connector:TestPoint") (at 247.65 142.24 180) (unit 1)
-    (in_bom yes) (on_board yes) (dnp no) (fields_autoplaced)
-    (property "Reference" "TP4" (at 250.19 144.907 0)
-      (effects (font (size 1.27 1.27)) (justify right))
-    )
-    (property "Value" "TestPoint" (at 250.19 147.447 0)
-      (effects (font (size 1.27 1.27)) (justify right))
-    )
-    (property "Footprint" "TestPoint:TestPoint_Pad_D1.0mm" (at 242.57 142.24 0)
-      (effects (font (size 1.27 1.27)) hide)
-    )
-    (property "Datasheet" "~" (at 242.57 142.24 0)
-      (effects (font (size 1.27 1.27)) hide)
-    )
-    (pin "1")
-    (instances
-      (project "pcb"
-        (path "/19e8f276-6a71-4fad-b0cb-92febe4a4ffd"
-          (reference "TP4") (unit 1)
-        )
-      )
-      (project "pcb"
-        (path "/20bda546-3b72-48f2-b51c-b61a4edfe0c6"
-          (reference "TP28") (unit 1)
-        )
-      )
-    )
-  )
   (symbol (lib_id "Device:R") (at 252.73 27.94 180) (unit 1)
     (in_bom yes) (on_board yes) (dnp no) (fields_autoplaced)
@@
     )
   )
-  (symbol (lib_id "Connector:TestPoint") (at 245.11 147.32 180) (unit 1)
-    (in_bom yes) (on_board yes) (dnp no) (fields_autoplaced)
-    (property "Reference" "TP3" (at 247.65 149.987 0)
-      (effects (font (size 1.27 1.27)) (justify right))
-    )
-    (property "Value" "TestPoint" (at 247.65 152.527 0)
-      (effects (font (size 1.27 1.27)) (justify right))
-    )
-    (property "Footprint" "TestPoint:TestPoint_Pad_D1.0mm" (at 240.03 147.32 0)
-      (effects (font (size 1.27 1.27)) hide)
-    )
-    (property "Datasheet" "~" (at 240.03 147.32 0)
-      (effects (font (size 1.27 1.27)) hide)
-    )
-    (pin "1")
-    (instances
-      (project "pcb"
-        (path "/19e8f276-6a71-4fad-b0cb-92febe4a4ffd"
-          (reference "TP3") (unit 1)
-        )
-      )
-      (project "pcb"
-        (path "/20bda546-3b72-48f2-b51c-b61a4edfe0c6"
-          (reference "TP27") (unit 1)
-        )
-      )
-    )
-  )
   (symbol (lib_id "DS4432U+:DS4432U+") (at 138.43 105.41 0) (unit 1)
     (in_bom yes) (on_board yes) (dnp no) (fields_autoplaced)
@@
     )
   )
+  (symbol (lib_id "Device:LED") (at 275.59 88.9 180) (unit 1)
+    (in_bom yes) (on_board yes) (dnp no) (fields_autoplaced)
+    (property "Reference" "D3" (at 277.1775 82.55 0)
+      (effects (font (size 1.27 1.27)))
+    )
+    (property "Value" "LED" (at 277.1775 85.09 0)
+      (effects (font (size 1.27 1.27)))
+    )
+    (property "Footprint" "LED_SMD:LED_0402_1005Metric" (at 275.59 88.9 0)
+      (effects (font (size 1.27 1.27)) hide)
+    )
+    (property "Datasheet" "~" (at 275.59 88.9 0)
+      (effects (font (size 1.27 1.27)) hide)
+    )
+    (property "LCSC" "C2856703" (at 275.59 88.9 0)
+      (effects (font (size 1.27 1.27)) hide)
+    )
+    (pin "1")
+    (pin "2")
+    (instances
+      (project "pcb"
+        (path "/20bda546-3b72-48f2-b51c-b61a4edfe0c6"
+          (reference "D3") (unit 1)
+        )
+      )
+    )
+  )
   (symbol (lib_id "Device:D_Schottky") (at 85.09 16.51 90) (unit 1)
     (in_bom yes) (on_board yes) (dnp no) (fields_autoplaced)
@@
         )
       )
+    )
+  )
+  (symbol (lib_id "power:GND") (at 242.57 154.94 180) (unit 1)
+    (in_bom yes) (on_board yes) (dnp no) (fields_autoplaced)
+    (property "Reference" "#PWR011" (at 242.57 148.59 0)
+      (effects (font (size 1.27 1.27)) hide)
+    )
+    (property "Value" "GND" (at 242.57 151.13 0)
+      (effects (font (size 1.27 1.27)))
+    )
+    (property "Footprint" "" (at 242.57 154.94 0)
+      (effects (font (size 1.27 1.27)) hide)
+    )
+    (property "Datasheet" "" (at 242.57 154.94 0)
+      (effects (font (size 1.27 1.27)) hide)
+    )
+    (pin "1")
+    (instances
+      (project "pcb"
+        (path "/20bda546-3b72-48f2-b51c-b61a4edfe0c6"
+          (reference "#PWR011") (unit 1)
+        )
+      )
+    )
+  )
+  (symbol (lib_id "Device:R") (at 283.21 88.9 90) (unit 1)
+    (in_bom yes) (on_board yes) (dnp no) (fields_autoplaced)
+    (property "Reference" "R11" (at 283.21 83.82 90)
+      (effects (font (size 1.27 1.27)))
+    )
+    (property "Value" "91" (at 283.21 86.36 90)
+      (effects (font (size 1.27 1.27)))
+    )
+    (property "Footprint" "Resistor_SMD:R_0402_1005Metric" (at 283.21 90.678 90)
+      (effects (font (size 1.27 1.27)) hide)
+    )
+    (property "Datasheet" "~" (at 283.21 88.9 0)
+      (effects (font (size 1.27 1.27)) hide)
+    )
+    (property "LCSC" "C2974023" (at 283.21 88.9 90)
+      (effects (font (size 1.27 1.27)) hide)
+    )
+    (pin "1")
+    (pin "2")
+    (instances
+      (project "pcb"
+        (path "/20bda546-3b72-48f2-b51c-b61a4edfe0c6"
+          (reference "R11") (unit 1)
+        )
+      )

Commit message: Update PCB
Parts:
- removed FPC1: THD0515-24CL-SN, THD0515-24CL-SN:FPC-SMD_24P-P0.50_THD0515-24CL-SN, symbol THD0515-24CL-SN:THD0515-24CL-SN
- removed R4: 10k, Resistor_SMD:R_0402_1005Metric, symbol Device:R
- removed TP2: TestPoint, TestPoint:TestPoint_Pad_1.0x1.0mm, symbol Connector:TestPoint
Changed lines of the file:
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@@
-    )
-  )
-  (symbol (lib_id "THD0515-24CL-SN:THD0515-24CL-SN") (at 200.66 30.48 0) (unit 1)
-    (in_bom yes) (on_board yes) (dnp no) (fields_autoplaced)
-    (property "Reference" "FPC1" (at 209.55 28.575 0)
-      (effects (font (size 1.27 1.27)) (justify left))
-    )
-    (property "Value" "THD0515-24CL-SN" (at 209.55 31.115 0)
-      (effects (font (size 1.27 1.27)) (justify left))
-    )
-    (property "Footprint" "THD0515-24CL-SN:FPC-SMD_24P-P0.50_THD0515-24CL-SN" (at 200.66 71.12 0)
-      (effects (font (size 1.27 1.27)) hide)
-    )
-    (property "Datasheet" "https://lcsc.com/product-detail/FFC-FPC-Flat-Flexible-Connectors_THD-THD0515-24CL-SN_C283150.html" (at 200.66 73.66 0)
-      (effects (font (size 1.27 1.27)) hide)
-    )
-    (property "LCSC Part" "C283150" (at 200.66 76.2 0)
-      (effects (font (size 1.27 1.27)) hide)
-    )
-    (pin "1")
-    (pin "10")
-    (pin "11")
-    (pin "12")
-    (pin "13")
-    (pin "14")
-    (pin "15")
-    (pin "16")
-    (pin "17")
-    (pin "18")
-    (pin "19")
-    (pin "2")
-    (pin "20")
-    (pin "21")
-    (pin "22")
-    (pin "23")
-    (pin "24")
-    (pin "25")
-    (pin "26")
-    (pin "3")
-    (pin "4")
-    (pin "5")
-    (pin "6")
-    (pin "7")
-    (pin "8")
-    (pin "9")
-    (instances
-      (project "pcb"
-        (path "/20bda546-3b72-48f2-b51c-b61a4edfe0c6"
-          (reference "FPC1") (unit 1)
-        )
-      )
     )
   )
@@
         (path "/20bda546-3b72-48f2-b51c-b61a4edfe0c6"
           (reference "#PWR035") (unit 1)
-        )
-      )
-    )
-  )
-  (symbol (lib_id "power:GND") (at 43.18 143.51 0) (unit 1)
-    (in_bom yes) (on_board yes) (dnp no) (fields_autoplaced)
-    (property "Reference" "#PWR017" (at 43.18 149.86 0)
-      (effects (font (size 1.27 1.27)) hide)
-    )
-    (property "Value" "GND" (at 43.18 148.59 0)
-      (effects (font (size 1.27 1.27)))
-    )
-    (property "Footprint" "" (at 43.18 143.51 0)
-      (effects (font (size 1.27 1.27)) hide)
-    )
-    (property "Datasheet" "" (at 43.18 143.51 0)
-      (effects (font (size 1.27 1.27)) hide)
-    )
-    (pin "1")
-    (instances
-      (project "pcb"
-        (path "/19e8f276-6a71-4fad-b0cb-92febe4a4ffd"
-          (reference "#PWR017") (unit 1)
-        )
-      )
-      (project "pcb"
-        (path "/20bda546-3b72-48f2-b51c-b61a4edfe0c6"
-          (reference "#PWR04") (unit 1)
         )
       )
@@
     )
   )
-  (symbol (lib_id "Connector:TestPoint") (at 43.18 143.51 90) (unit 1)
-    (in_bom yes) (on_board yes) (dnp no) (fields_autoplaced)
-    (property "Reference" "TP2" (at 39.878 138.43 90)
-      (effects (font (size 1.27 1.27)))
-    )
-    (property "Value" "TestPoint" (at 39.878 140.97 90)
-      (effects (font (size 1.27 1.27)))
-    )
-    (property "Footprint" "TestPoint:TestPoint_Pad_1.0x1.0mm" (at 43.18 138.43 0)
-      (effects (font (size 1.27 1.27)) hide)
-    )
-    (property "Datasheet" "~" (at 43.18 138.43 0)
-      (effects (font (size 1.27 1.27)) hide)
-    )
-    (pin "1")
-    (instances
-      (project "pcb"
-        (path "/19e8f276-6a71-4fad-b0cb-92febe4a4ffd"
-          (reference "TP2") (unit 1)
-        )
-      )
-      (project "pcb"
-        (path "/20bda546-3b72-48f2-b51c-b61a4edfe0c6"
-          (reference "TP2") (unit 1)
-        )
-      )
-    )
-  )
   (symbol (lib_id "power:+1V1") (at 240.03 40.64 0) (unit 1)
     (in_bom yes) (on_board yes) (dnp no) (fields_autoplaced)
@@
         )
       )
-    )
-  )
-  (symbol (lib_id "Device:R") (at 21.59 153.67 0) (unit 1)
-    (in_bom yes) (on_board yes) (dnp no) (fields_autoplaced)
-    (property "Reference" "R4" (at 24.13 153.035 0)
-      (effects (font (size 1.27 1.27)) (justify left))
-    )
-    (property "Value" "10k" (at 24.13 155.575 0)
-      (effects (font (size 1.27 1.27)) (justify left))
-    )
-    (property "Footprint" "Resistor_SMD:R_0402_1005Metric" (at 19.812 153.67 90)
-      (effects (font (size 1.27 1.27)) hide)
-    )
-    (property "Datasheet" "~" (at 21.59 153.67 0)
-      (effects (font (size 1.27 1.27)) hide)
-    )
-    (property "LCSC" "C2991755" (at 21.59 153.67 0)
-      (effects (font (size 1.27 1.27)) hide)
-    )
-    (pin "1")
-    (pin "2")
-    (instances
-      (project "pcb"
-        (path "/19e8f276-6a71-4fad-b0cb-92febe4a4ffd"
-          (reference "R4") (unit 1)
-        )
-      )
-      (project "pcb"
-        (path "/20bda546-3b72-48f2-b51c-b61a4edfe0c6"
-          (reference "R1") (unit 1)
-        )
-      )
