File: pcb/pcb.kicad_sch (KiCad schematic)
At the start: 45 parts, among them J1 Conn_01x01_Socket, J2 Conn_01x02_Socket, J3 Conn_01x02_Socket, J4 Conn_01x01_Socket, K1 G3VM-31WR_TR05_, U1 AP2112K-3.3TRG1, U2 W25Q16JVUXIQ, U3 RP2040, U4 DS4432U+T&amp;R, U5 AD8403ARUZ1-REEL, Y2 Crystal_GND24_Small

Commit message: wip
Parts:
- removed J1, J4: Conn_01x01_Socket, Connector_PinSocket_2.54mm:PinSocket_1x01_P2.54mm_Vertical, symbol Connector:Conn_01x01_Socket
- removed J2, J3: Conn_01x02_Socket, Connector_PinSocket_2.54mm:PinSocket_1x02_P2.54mm_Vertical, symbol Connector:Conn_01x02_Socket
- added J1: Conn_01x02_Socket, Connector_PinSocket_2.54mm:PinSocket_1x02_P2.54mm_Vertical, symbol Connector:Conn_01x02_Socket
- added J2: Conn_01x04_Socket, Connector_PinSocket_2.54mm:PinSocket_1x04_P2.54mm_Vertical, symbol Connector:Conn_01x04_Socket
Connections:
- net GND: now also J1.1 (Pin_1)
- net UART_TX: now reaches U3.2 (GPIO0)
- net UART_TX: now also J2.1 (Pin_1)
- net at U3.24 (SWCLK): now also J2.3 (Pin_3)
- net at U3.25 (SWD): now also J2.4 (Pin_4)
- net UART_RX: now reaches U3.3 (GPIO1)
- net UART_RX: now also J2.2 (Pin_2)
- net at R3.1: now also J1.2 (Pin_2)
Changed lines of the file:
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@@
     (stroke (width 0) (type default))
   )
-  (wire (pts (xy 167.64 130.81) (xy 173.99 130.81))
+  (wire (pts (xy 162.56 130.81) (xy 173.99 130.81))
     (stroke (width 0) (type default))
   )
@@
     (stroke (width 0) (type default))
   )
-  (wire (pts (xy 167.64 133.35) (xy 173.99 133.35))
+  (wire (pts (xy 162.56 133.35) (xy 173.99 133.35))
     (stroke (width 0) (type default))
   )
@@
     )
   )
+  (global_label "UART_TX" (shape input) (at 162.56 125.73 0) (fields_autoplaced)
+    (effects (font (size 1.27 1.27)) (justify left))
+    (property "Intersheetrefs" "${INTERSHEET_REFS}" (at 173.2672 125.73 0)
+      (effects (font (size 1.27 1.27)) (justify left) hide)
+    )
+  )
   (global_label "3DS_TP32_5V" (shape input) (at 81.28 27.94 180) (fields_autoplaced)
     (effects (font (size 1.27 1.27)) (justify right))
@@
     )
   )
+  (global_label "UART_RX" (shape input) (at 237.49 68.58 0) (fields_autoplaced)
+    (effects (font (size 1.27 1.27)) (justify left))
+    (property "Intersheetrefs" "${INTERSHEET_REFS}" (at 248.4996 68.58 0)
+      (effects (font (size 1.27 1.27)) (justify left) hide)
+    )
+  )
   (global_label "3DS_TP52_POWER" (shape input) (at 134.62 158.75 0) (fields_autoplaced)
     (effects (font (size 1.27 1.27)) (justify left))
@@
     (property "Intersheetrefs" "${INTERSHEET_REFS}" (at 40.3951 137.16 0)
       (effects (font (size 1.27 1.27)) (justify right) hide)
+    )
+  )
+  (global_label "UART_RX" (shape input) (at 162.56 128.27 0) (fields_autoplaced)
+    (effects (font (size 1.27 1.27)) (justify left))
+    (property "Intersheetrefs" "${INTERSHEET_REFS}" (at 173.5696 128.27 0)
+      (effects (font (size 1.27 1.27)) (justify left) hide)
+    )
+  )
+  (global_label "UART_TX" (shape input) (at 237.49 66.04 0) (fields_autoplaced)
+    (effects (font (size 1.27 1.27)) (justify left))
+    (property "Intersheetrefs" "${INTERSHEET_REFS}" (at 248.1972 66.04 0)
+      (effects (font (size 1.27 1.27)) (justify left) hide)
     )
   )
@@
     )
   )
-  (symbol (lib_id "power:GND") (at 167.64 139.7 0) (unit 1)
-    (in_bom yes) (on_board yes) (dnp no) (fields_autoplaced)
-    (property "Reference" "#PWR029" (at 167.64 146.05 0)
-      (effects (font (size 1.27 1.27)) hide)
-    )
-    (property "Value" "GND" (at 167.64 144.78 0)
-      (effects (font (size 1.27 1.27)))
-    )
-    (property "Footprint" "" (at 167.64 139.7 0)
-      (effects (font (size 1.27 1.27)) hide)
-    )
-    (property "Datasheet" "" (at 167.64 139.7 0)
-      (effects (font (size 1.27 1.27)) hide)
-    )
-    (pin "1")
-    (instances
-      (project "pcb"
-        (path "/4db5c0ae-dab5-4243-9886-99aa858b7752"
-          (reference "#PWR029") (unit 1)
-        )
-      )
-    )
-  )
   (symbol (lib_id "Device:C_Small") (at 238.76 34.29 0) (unit 1)
     (in_bom yes) (on_board yes) (dnp no) (fields_autoplaced)
@@
         (path "/4db5c0ae-dab5-4243-9886-99aa858b7752"
           (reference "#PWR032") (unit 1)
-        )
-      )
-    )
-  )
-  (symbol (lib_id "Connector:Conn_01x01_Socket") (at 162.56 139.7 180) (unit 1)
-    (in_bom yes) (on_board yes) (dnp no) (fields_autoplaced)
-    (property "Reference" "J4" (at 163.195 135.89 0)
-      (effects (font (size 1.27 1.27)))
-    )
-    (property "Value" "Conn_01x01_Socket" (at 163.195 138.43 0)
-      (effects (font (size 1.27 1.27)))
-    )
-    (property "Footprint" "Connector_PinSocket_2.54mm:PinSocket_1x01_P2.54mm_Vertical" (at 162.56 139.7 0)
-      (effects (font (size 1.27 1.27)) hide)
-    )
-    (property "Datasheet" "~" (at 162.56 139.7 0)
-      (effects (font (size 1.27 1.27)) hide)
-    )
-    (pin "1")
-    (instances
-      (project "pcb"
-        (path "/4db5c0ae-dab5-4243-9886-99aa858b7752"
-          (reference "J4") (unit 1)
         )
       )
@@
     )
   )
+  (symbol (lib_id "Connector:Conn_01x04_Socket") (at 157.48 128.27 0) (mirror y) (unit 1)
+    (in_bom yes) (on_board yes) (dnp no) (fields_autoplaced)
+    (property "Reference" "J2" (at 158.115 121.92 0)
+      (effects (font (size 1.27 1.27)))
+    )
+    (property "Value" "Conn_01x04_Socket" (at 158.115 124.46 0)
+      (effects (font (size 1.27 1.27)))
+    )
+    (property "Footprint" "Connector_PinSocket_2.54mm:PinSocket_1x04_P2.54mm_Vertical" (at 157.48 128.27 0)
+      (effects (font (size 1.27 1.27)) hide)
+    )
+    (property "Datasheet" "~" (at 157.48 128.27 0)
+      (effects (font (size 1.27 1.27)) hide)
+    )
+    (pin "1")
+    (pin "2")
+    (pin "3")
+    (pin "4")
+    (instances
+      (project "pcb"
+        (path "/4db5c0ae-dab5-4243-9886-99aa858b7752"
+          (reference "J2") (unit 1)
+        )
+      )
+    )
+  )
   (symbol (lib_id "Device:R_Small") (at 92.71 144.78 90) (unit 1)
     (in_bom yes) (on_board yes) (dnp no) (fields_autoplaced)
@@
         (path "/4db5c0ae-dab5-4243-9886-99aa858b7752"
           (reference "#PWR038") (unit 1)
-        )
-      )
-    )
-  )
-  (symbol (lib_id "Connector:Conn_01x01_Socket") (at 72.39 50.8 90) (unit 1)
-    (in_bom yes) (on_board yes) (dnp no) (fields_autoplaced)
-    (property "Reference" "J1" (at 73.66 50.8 90)
-      (effects (font (size 1.27 1.27)) (justify right))
-    )
-    (property "Value" "Conn_01x01_Socket" (at 73.66 53.34 90)
-      (effects (font (size 1.27 1.27)) (justify right))
-    )
-    (property "Footprint" "Connector_PinSocket_2.54mm:PinSocket_1x01_P2.54mm_Vertical" (at 72.39 50.8 0)
-      (effects (font (size 1.27 1.27)) hide)
-    )
-    (property "Datasheet" "~" (at 72.39 50.8 0)
-      (effects (font (size 1.27 1.27)) hide)
-    )
-    (pin "1")
-    (instances
-      (project "pcb"
-        (path "/4db5c0ae-dab5-4243-9886-99aa858b7752"
-          (reference "J1") (unit 1)
         )
       )
@@
         (path "/4db5c0ae-dab5-4243-9886-99aa858b7752"
           (reference "#PWR06") (unit 1)
-        )
-      )
-    )
-  )
-  (symbol (lib_id "Connector:Conn_01x02_Socket") (at 242.57 66.04 0) (unit 1)
-    (in_bom yes) (on_board yes) (dnp no)
-    (property "Reference" "J3" (at 243.84 66.04 0)
-      (effects (font (size 1.27 1.27)) (justify left))
-    )
-    (property "Value" "Conn_01x02_Socket" (at 243.84 68.58 0)
-      (effects (font (size 1.27 1.27)) (justify left))
-    )
-    (property "Footprint" "Connector_PinSocket_2.54mm:PinSocket_1x02_P2.54mm_Vertical" (at 242.57 66.04 0)
-      (effects (font (size 1.27 1.27)) hide)
-    )
-    (property "Datasheet" "~" (at 242.57 66.04 0)
-      (effects (font (size 1.27 1.27)) hide)
-    )
-    (pin "1")
-    (pin "2")
-    (instances
-      (project "pcb"
-        (path "/4db5c0ae-dab5-4243-9886-99aa858b7752"
-          (reference "J3") (unit 1)
         )
       )
@@
     )
   )
-  (symbol (lib_id "Connector:Conn_01x02_Socket") (at 162.56 130.81 0) (mirror y) (unit 1)
-    (in_bom yes) (on_board yes) (dnp no) (fields_autoplaced)
-    (property "Reference" "J2" (at 163.195 127 0)
-      (effects (font (size 1.27 1.27)))
-    )
-    (property "Value" "Conn_01x02_Socket" (at 163.195 129.54 0)
-      (effects (font (size 1.27 1.27)))
-    )
-    (property "Footprint" "Connector_PinSocket_2.54mm:PinSocket_1x02_P2.54mm_Vertical" (at 162.56 130.81 0)
-      (effects (font (size 1.27 1.27)) hide)
-    )
-    (property "Datasheet" "~" (at 162.56 130.81 0)
-      (effects (font (size 1.27 1.27)) hide)
-    )
-    (pin "1")
-    (pin "2")
-    (instances
-      (project "pcb"
-        (path "/4db5c0ae-dab5-4243-9886-99aa858b7752"
-          (reference "J2") (unit 1)
-        )
-      )
-    )
-  )
   (symbol (lib_id "Device:C_Small") (at 170.18 34.29 0) (mirror x) (unit 1)
     (in_bom yes) (on_board yes) (dnp no)
@@
     )
   )
+  (symbol (lib_id "power:GND") (at 69.85 55.88 0) (unit 1)
+    (in_bom yes) (on_board yes) (dnp no) (fields_autoplaced)
+    (property "Reference" "#PWR040" (at 69.85 62.23 0)
+      (effects (font (size 1.27 1.27)) hide)
+    )
+    (property "Value" "GND" (at 69.85 60.96 0)
+      (effects (font (size 1.27 1.27)))
+    )
+    (property "Footprint" "" (at 69.85 55.88 0)
+      (effects (font (size 1.27 1.27)) hide)
+    )
+    (property "Datasheet" "" (at 69.85 55.88 0)
+      (effects (font (size 1.27 1.27)) hide)
+    )
+    (pin "1")
+    (instances
+      (project "pcb"
+        (path "/4db5c0ae-dab5-4243-9886-99aa858b7752"
+          (reference "#PWR040") (unit 1)
+        )
+      )
+    )
+  )
   (symbol (lib_id "Device:C_Small") (at 86.36 160.02 0) (unit 1)
     (in_bom yes) (on_board yes) (dnp no)
@@
         )
       )
+    )
+  )
+  (symbol (lib_id "Connector:Conn_01x02_Socket") (at 69.85 50.8 90) (unit 1)
+    (in_bom yes) (on_board yes) (dnp no) (fields_autoplaced)
+    (property "Reference" "J1" (at 73.66 50.8 90)
+      (effects (font (size 1.27 1.27)) (justify right))
+    )
+    (property "Value" "Conn_01x02_Socket" (at 73.66 53.34 90)
+      (effects (font (size 1.27 1.27)) (justify right))
+    )
+    (property "Footprint" "Connector_PinSocket_2.54mm:PinSocket_1x02_P2.54mm_Vertical" (at 69.85 50.8 0)
+      (effects (font (size 1.27 1.27)) hide)
+    )
+    (property "Datasheet" "~" (at 69.85 50.8 0)
+      (effects (font (size 1.27 1.27)) hide)
+    )
+    (pin "1")
+    (pin "2")
+    (instances
+      (project "pcb"
+        (path "/4db5c0ae-dab5-4243-9886-99aa858b7752"
+          (reference "J1") (unit 1)
+        )
+      )

Commit message: pcb
Parts:
- removed K1: G3VM-31WR_TR05_, G3VM-31WR_TR05_:G3VM-31WR_TR05_, symbol G3VM-31WR_TR05_:G3VM-31WR_TR05_
- removed R10: 430, Resistor_SMD:R_0402_1005Metric, symbol Device:R_Small
- added C19: 100n, Capacitor_SMD:C_0402_1005Metric, symbol Device:C_Small
- added U6: ADG801BRTZ-REEL7, ADG801BRTZ-REEL7:SOT-23-6_L2.9-W1.6-P0.95-LS2.8-BL, symbol ADG801BRTZ-REEL7:ADG801BRTZ-REEL7
- Y2: footprint Crystal:Crystal_SMD_2520-4Pin_2.5x2.0mm -> Crystal:Crystal_SMD_3225-4Pin_3.2x2.5mm
Connections:
- net +3V3: now also C19.1, U6.6 (VDD)
- net GND: now also C19.2, U6.3 (GND); no longer FPC1.25, FPC1.26
- net RELAY_A: now also U6.4 (IN)
- net at U5.4 (W2): now also U6.2 (S)
- net at U5.8 (W4): now also U6.1 (D)
- no-connect marks 11 -> 14

Commit message: flex
Parts:
- added TP1: TestPoint, TestPoint:TestPoint_Pad_D1.5mm, symbol Connector:TestPoint
Connections:
- net 3DS_TP32_5V: now also TP1.1
- net USB_D-: now reaches R6.1, U3.46 (USB_DM)
- net USB_D+: now reaches R5.1, U3.47 (USB_DP)
Other:
- moved on the sheet: R5, R6
Changed lines of the file:
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@@
+    (stroke (width 0) (type default))
+  )
+  (wire (pts (xy 245.11 55.88) (xy 237.49 55.88))
     (stroke (width 0) (type default))
   )
@@
     (stroke (width 0) (type default))
   )
+  (wire (pts (xy 237.49 58.42) (xy 245.11 58.42))
+    (stroke (width 0) (type default))
+  )
   (wire (pts (xy 45.72 44.45) (xy 45.72 43.18))
     (stroke (width 0) (type default))
@@
     (stroke (width 0) (type default))
   )
+  (wire (pts (xy 80.01 27.94) (xy 81.28 27.94))
+    (stroke (width 0) (type default))
+  )
   (wire (pts (xy 182.88 25.4) (xy 182.88 31.75))
     (stroke (width 0) (type default))
@@
     (stroke (width 0) (type default))
   )
+  (wire (pts (xy 80.01 34.29) (xy 80.01 27.94))
+    (stroke (width 0) (type default))
+  )
   (wire (pts (xy 33.02 58.42) (xy 35.56 58.42))
     (stroke (width 0) (type default))
@@
   )
   (text "Not assigned to CS, a normal GPIO." (at 247.65 116.84 0)
+    (effects (font (size 1.27 1.27)) (justify left bottom))
+  )
+  (label "USB_D-" (at 237.49 58.42 0) (fields_autoplaced)
+    (effects (font (size 1.27 1.27)) (justify left bottom))
+  )
+  (label "USB_D+" (at 237.49 55.88 0) (fields_autoplaced)
     (effects (font (size 1.27 1.27)) (justify left bottom))
   )
@@
     )
   )
-  (global_label "3DS_TP32_5V" (shape input) (at 81.28 27.94 180) (fields_autoplaced)
+  (global_label "3DS_TP32_5V" (shape input) (at 80.01 27.94 180) (fields_autoplaced)
     (effects (font (size 1.27 1.27)) (justify right))
-    (property "Intersheetrefs" "${INTERSHEET_REFS}" (at 65.7953 27.94 0)
+    (property "Intersheetrefs" "${INTERSHEET_REFS}" (at 64.5253 27.94 0)
       (effects (font (size 1.27 1.27)) (justify right) hide)
     )
@@
     )
   )
-  (global_label "D-" (shape input) (at 245.11 58.42 0) (fields_autoplaced)
-    (effects (font (size 1.27 1.27)) (justify left))
-    (property "Intersheetrefs" "${INTERSHEET_REFS}" (at 250.8582 58.42 0)
+  (global_label "D-" (shape input) (at 252.73 58.42 0) (fields_autoplaced)
+    (effects (font (size 1.27 1.27)) (justify left))
+    (property "Intersheetrefs" "${INTERSHEET_REFS}" (at 258.4782 58.42 0)
       (effects (font (size 1.27 1.27)) (justify left) hide)
     )
@@
     )
   )
-  (global_label "D+" (shape input) (at 245.11 55.88 0) (fields_autoplaced)
-    (effects (font (size 1.27 1.27)) (justify left))
-    (property "Intersheetrefs" "${INTERSHEET_REFS}" (at 250.8582 55.88 0)
+  (global_label "D+" (shape input) (at 252.73 55.88 0) (fields_autoplaced)
+    (effects (font (size 1.27 1.27)) (justify left))
+    (property "Intersheetrefs" "${INTERSHEET_REFS}" (at 258.4782 55.88 0)
       (effects (font (size 1.27 1.27)) (justify left) hide)
     )
@@
     )
   )
-  (symbol (lib_id "Device:R") (at 241.3 55.88 90) (unit 1)
-    (in_bom yes) (on_board yes) (dnp no) (fields_autoplaced)
-    (property "Reference" "R5" (at 241.3 50.8 90)
-      (effects (font (size 1.27 1.27)))
-    )
-    (property "Value" "27" (at 241.3 53.34 90)
-      (effects (font (size 1.27 1.27)))
-    )
-    (property "Footprint" "Resistor_SMD:R_0402_1005Metric" (at 241.3 57.658 90)
-      (effects (font (size 1.27 1.27)) hide)
-    )
-    (property "Datasheet" "~" (at 241.3 55.88 0)
-      (effects (font (size 1.27 1.27)) hide)
-    )
-    (property "LCSC" "C102938" (at 241.3 55.88 90)
+  (symbol (lib_id "Device:R") (at 248.92 55.88 90) (unit 1)
+    (in_bom yes) (on_board yes) (dnp no) (fields_autoplaced)
+    (property "Reference" "R5" (at 248.92 50.8 90)
+      (effects (font (size 1.27 1.27)))
+    )
+    (property "Value" "27" (at 248.92 53.34 90)
+      (effects (font (size 1.27 1.27)))
+    )
+    (property "Footprint" "Resistor_SMD:R_0402_1005Metric" (at 248.92 57.658 90)
+      (effects (font (size 1.27 1.27)) hide)
+    )
+    (property "Datasheet" "~" (at 248.92 55.88 0)
+      (effects (font (size 1.27 1.27)) hide)
+    )
+    (property "LCSC" "C102938" (at 248.92 55.88 90)
       (effects (font (size 1.27 1.27)) hide)
     )
@@
         (path "/4db5c0ae-dab5-4243-9886-99aa858b7752"
           (reference "R11") (unit 1)
+        )
+      )
+    )
+  )
+  (symbol (lib_id "Connector:TestPoint") (at 80.01 34.29 180) (unit 1)
+    (in_bom yes) (on_board yes) (dnp no) (fields_autoplaced)
+    (property "Reference" "TP1" (at 82.55 36.957 0)
+      (effects (font (size 1.27 1.27)) (justify right))
+    )
+    (property "Value" "TestPoint" (at 82.55 39.497 0)
+      (effects (font (size 1.27 1.27)) (justify right))
+    )
+    (property "Footprint" "TestPoint:TestPoint_Pad_D1.5mm" (at 74.93 34.29 0)
+      (effects (font (size 1.27 1.27)) hide)
+    )
+    (property "Datasheet" "~" (at 74.93 34.29 0)
+      (effects (font (size 1.27 1.27)) hide)
+    )
+    (pin "1")
+    (instances
+      (project "pcb"
+        (path "/4db5c0ae-dab5-4243-9886-99aa858b7752"
+          (reference "TP1") (unit 1)
         )
       )
@@
     )
   )
-  (symbol (lib_id "Device:R") (at 241.3 58.42 90) (mirror x) (unit 1)
+  (symbol (lib_id "Device:R") (at 248.92 58.42 90) (mirror x) (unit 1)
     (in_bom yes) (on_board yes) (dnp no)
-    (property "Reference" "R6" (at 241.3 63.5 90)
-      (effects (font (size 1.27 1.27)))
-    )
-    (property "Value" "27" (at 241.3 60.96 90)
-      (effects (font (size 1.27 1.27)))
-    )
-    (property "Footprint" "Resistor_SMD:R_0402_1005Metric" (at 241.3 56.642 90)
-      (effects (font (size 1.27 1.27)) hide)
-    )
-    (property "Datasheet" "~" (at 241.3 58.42 0)
-      (effects (font (size 1.27 1.27)) hide)
-    )
-    (property "LCSC" "C102938" (at 241.3 58.42 90)
-      (effects (font (size 1.27 1.27)) hide)
-    )
+    (property "Reference" "R6" (at 248.92 63.5 90)
+      (effects (font (size 1.27 1.27)))
+    )
+    (property "Value" "27" (at 248.92 60.96 90)
+      (effects (font (size 1.27 1.27)))
+    )
+    (property "Footprint" "Resistor_SMD:R_0402_1005Metric" (at 248.92 56.642 90)
+      (effects (font (size 1.27 1.27)) hide)
+    )
+    (property "Datasheet" "~" (at 248.92 58.42 0)
+      (effects (font (size 1.27 1.27)) hide)
+    )
+    (property "LCSC" "C102938" (at 248.92 58.42 90)
+      (effects (font (size 1.27 1.27)) hide)
+    )
