File: flex/flex_xl/flex_xl.kicad_sch (KiCad schematic)
At the start: 2 parts, among them J2 Conn_01x24_Pin

Commit message: Change footprint name
Parts:
- e1: footprint 3DS_LL:3DS_LL -> 3ds_xl:3ds_xl
Changed lines of the file:
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@@
       (effects (font (size 1.27 1.27)))
     )
-    (property "Footprint" "3DS_LL:3DS_LL" (at 71.12 78.74 0)
+    (property "Footprint" "3ds_xl:3ds_xl" (at 71.12 78.74 0)
       (effects (font (size 1.27 1.27)) hide)
     )
@@
     (pin "9")
     (instances
-      (project "flex"
+      (project "flex_xl"
         (path "/9ae2b03a-48a0-445d-83ec-edfc9c6f4ccc"
           (reference "e1") (unit 1)
@@
     (pin "9")
     (instances
-      (project "flex"
+      (project "flex_xl"
         (path "/9ae2b03a-48a0-445d-83ec-edfc9c6f4ccc"
           (reference "J2") (unit 1)
