File: pcb/fastener/fastener.kicad_pcb (KiCad board)
At the start: 2 copper layers, 20.7 x 32.1 mm, 12 parts

Commit message: Update flex order detail
Parts:
- removed the REF** at (51.0, 95.7)
- removed the REF** at (68.2, 80.2)
- removed the REF** at (59.5, 78.5)
- removed the REF** at (51.0, 80.2)
- removed the REF** at (68.2, 95.7)
- removed the REF** at (67.3, 73.7)
- removed the REF** at (63.4, 87.9)
- removed the REF** at (51.9, 73.7)
- removed the REF** at (51.8, 102.2)
- removed the REF** at (67.2, 102.2)
- removed the REF** at (55.7, 88.0)
- added REF**: MouseBites_2.54, MouseBites:MouseBites_2.54, F.Cu at (70.0, 86.9)
- added REF**: MountingHole_2.2mm_M2_ISO7380, MountingHole:MountingHole_2.2mm_M2_ISO7380, F.Cu at (67.7, 102.0)
- added REF**: MouseBites_2.54, MouseBites:MouseBites_2.54, F.Cu at (59.5, 76.5)
- added REF**: MountingHole_2.2mm_M2_ISO7380, MountingHole:MountingHole_2.2mm_M2_ISO7380, F.Cu at (51.3, 71.9)
- added REF**: MouseBites_2.54, MouseBites:MouseBites_2.54, F.Cu at (49.0, 87.0)
- added REF**: MountingHole_2.2mm_M2_ISO7380, MountingHole:MountingHole_2.2mm_M2_ISO7380, F.Cu at (44.5, 95.2)
- added REF**: MountingHole_2.2mm_M2_ISO7380, MountingHole:MountingHole_2.2mm_M2_ISO7380, F.Cu at (44.5, 78.8)
- added REF**: MountingHole_2.2mm_M2_ISO7380, MountingHole:MountingHole_2.2mm_M2_ISO7380, F.Cu at (74.5, 95.2)
- added REF**: MountingHole_2.2mm_M2_ISO7380, MountingHole:MountingHole_2.2mm_M2_ISO7380, F.Cu at (74.5, 78.8)
- added REF**: MountingHole_2.2mm_M2_ISO7380, MountingHole:MountingHole_2.2mm_M2_ISO7380, F.Cu at (51.3, 102.0)
- added REF**: MountingHole_2.2mm_M2_ISO7380, MountingHole:MountingHole_2.2mm_M2_ISO7380, F.Cu at (67.7, 71.9)
Other:
- board size 20.7 x 32.1 mm -> 34.1 x 34.1 mm
